Commit message: RViz visualizations + joint control

File: spot_urdf/urdf/spot.urdf (robot description, URDF)
Before this commit: robot spot, 13 links, 12 joints
Links:
- removed link base
- added link base_link; visual mesh filename=package://spot_urdf/link_models/base.stl
- link fl.hip: geometry visual mesh filename=package://spot_urdf/link_models/fl.hip.stl
- link fl.lleg: geometry visual mesh filename=package://spot_urdf/link_models/fl.lleg.stl
- link fl.uleg: geometry visual mesh filename=package://spot_urdf/link_models/fl.uleg.stl
- link fr.hip: geometry visual mesh filename=package://spot_urdf/link_models/fr.hip.stl
- link fr.lleg: geometry visual mesh filename=package://spot_urdf/link_models/fr.lleg.stl
- link fr.uleg: geometry visual mesh filename=package://spot_urdf/link_models/fr.uleg.stl
- link hl.hip: geometry visual mesh filename=package://spot_urdf/link_models/hl.hip.stl
- link hl.lleg: geometry visual mesh filename=package://spot_urdf/link_models/hl.lleg.stl
- link hl.uleg: geometry visual mesh filename=package://spot_urdf/link_models/hl.uleg.stl
- link hr.hip: geometry visual mesh filename=package://spot_urdf/link_models/hr.hip.stl
- link hr.lleg: geometry visual mesh filename=package://spot_urdf/link_models/hr.lleg.stl
- link hr.uleg: geometry visual mesh filename=package://spot_urdf/link_models/hr.uleg.stl
Joints:
- joint fl.hx: parent base -> base_link
- joint fr.hx: parent base -> base_link
- joint hl.hx: parent base -> base_link
- joint hr.hx: parent base -> base_link
